File: Eagel/SchemaRobotV1.0.brd (EAGLE design)
At the start: 160 x 100 mm, 24 parts

Commit message: eagle
update schema
Parts:
- removed SV1: (no value), con-amp-mt:L11P
- removed SV3, SV4, SV5: (no value), con-amp-mt:L05P
- removed SV6: (no value), con-amp-mt:L08P
- removed SV7: (no value), con-amp-mt:L02P
- added J1, J2, J3, J5: (no value), SparkFun-Connectors:SCREWTERMINAL-3.5MM-4
- added J4, J6: (no value), SparkFun-Connectors:SCREWTERMINAL-3.5MM-8
- added J7: (no value), SparkFun-Connectors:SCREWTERMINAL-3.5MM-2
Connections:
- net ECHO: now also J1.3, J2.3, J3.3; no longer SV3.2, SV4.2, SV5.2
- net ENA: now also J4.8; no longer SV6.1
- net ENB: now also J4.3; no longer SV6.6
- net GND: now also J1.1, J2.1, J3.1, J4.2, J5.1; no longer SV1.11, SV3.5, SV4.5, SV5.5, SV6.7
- net IN1: now also J4.7; no longer SV6.2
- net IN2: now also J4.6; no longer SV6.3
- net IN3: now also J4.5; no longer SV6.4
- net IN4: now also J4.4; no longer SV6.5
- net IRS: now also J6.6; no longer SV1.5
- net IRS1: now also J6.8; no longer SV1.3
- net IRS2: now also J6.7; no longer SV1.4
- net IRS4: now also J6.5; no longer SV1.6
- net IRS6: now also J6.3; no longer SV1.8
- net IRS7: now also J6.2; no longer SV1.9
- net IRS8: now also J6.1; no longer SV1.10
- net LEDON: now also J5.2; no longer SV1.2
- net N$13: now also J7.2; no longer SV7.1
- net N$14: now also J7.1; no longer SV7.2
- net N$21: now also J6.4; no longer SV1.7
- net TRIG: now also J1.2, J2.2, J3.2; no longer SV3.3, SV4.3, SV5.3
- net VCC: now also J1.4, J2.4, J3.4, J4.1, J5.3; no longer SV1.1, SV3.1, SV4.1, SV5.1, SV6.8

Commit message: eagle
connectoren vervangen
Parts:
- moved J7 311.8 mm to (97.8, 85.1)
- moved J6 303.8 mm to (120.7, 88.9)
- moved J3 246.2 mm to (144.8, 72.4)
- moved J4 245.8 mm to (104.1, 73.7)
- moved J5 238.9 mm to (144.8, 22.9)
- moved J2 217.8 mm to (143.5, 58.4)
- moved J1 192.2 mm to (141.0, 47.0)

Commit message: eagle
schema bijna af!
Parts:
- removed C1, C2: (no value), rcl:C025-024X044
- removed Q1: (no value), special:Q
- removed S2: (no value), switch-dil:DS-01
- removed SV8: (no value), con-amp-mt:L16P
- added J8: Connector LCD, SparkFun-Connectors:1X20
- added S4: (no value), SparkFun-Switches:SWITCH_SPDT_PTH_11.6X4.0MM
- J1: value (none) -> Connector US1
- J2, J3: value (none) -> Connector US 2
- J4: value (none) -> Connector H-Brug
- J5: value (none) -> Connector IR voeding
- J6: value (none) -> Connector IR signalen
- J7: value (none) -> Connector batterij 12v
- R1, R2, R3, R4, R5: value (none) -> 100 ohm
- moved S3 134.7 mm to (129.0, 12.8), turned to 270 degrees
- moved J7 86.9 mm to (130.7, 4.61), turned to 180 degrees
- moved J6 84.1 mm to (114.3, 5.08), turned to 180 degrees
- moved S1 77.1 mm to (61.6, 10.9), turned to 180 degrees
- moved J3 71.0 mm to (73.8, 74.9)
- moved J4 68.3 mm to (35.8, 74.9)
- moved J5 61.1 mm to (86.4, 5.08), turned to 180 degrees
- moved J2 58.1 mm to (87.8, 74.9)
- moved J1 48.2 mm to (101.7, 74.9)
- moved LED1 8.87 mm to (11.1, 14.0)
- moved LED2 8.07 mm to (17.7, 14.0)
- moved LED3 7.32 mm to (24.3, 14.0)
- moved R1 7.27 mm to (11.1, 6.35)
- moved LED4 6.64 mm to (30.9, 14.0)
- moved R2 6.27 mm to (17.7, 6.35)
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Connections:
- removed net ECHO: DEVICE1.P1.0/SWDIO, DEVICE1.P12.1/I2C(SDA), DEVICE1.P12.3, J1.3, J2.3, J3.3
- removed net IRS: DEVICE1.P2.3, J6.6
- removed net N$15: DEVICE1.P0.1, SV8.13
- removed net N$16: DEVICE1.P0.0, SV8.14
- removed net N$17: C1.1, DEVICE1.P15.2/XTAL_OUT, Q1.1
- removed net N$18: C2.1, DEVICE1.P15.3/XTAL_IN, Q1.2
- removed net N$21: J6.4
- removed net TRIG: DEVICE1.P1.1/SWDCLK, DEVICE1.P12.0/I2C(SCL), DEVICE1.P12.2, J1.2, J2.2, J3.2
- new net ECHO1: DEVICE1.P12.3, J1.3
- new net ECHO2: DEVICE1.P12.1/I2C(SDA), J2.3
- new net ECHO3: DEVICE1.P1.0/SWDIO, J3.3
- new net IRS3: DEVICE1.P0.5, J6.3
- new net IRS5: DEVICE1.P0.3/EXT_REF0, J6.5
- new net N$1: DEVICE1.P2.3, J8.14
- new net N$7: DEVICE1.P2.2/SW1, J8.13
- new net TRIG1: DEVICE1.P12.2, J1.2
- new net TRIG2: DEVICE1.P12.0/I2C(SCL), J2.2
- new net TRIG3: DEVICE1.P1.1/SWDCLK, J3.2
- net GND: now also J5.3, J5.4, J8.1, J8.3, S4.3; no longer C1.2, C2.2, J5.1, SV8.1, SV8.3
- net IRS1: now also DEVICE1.P0.7, J6.1; no longer DEVICE1.P2.1/LED1, J6.8
- net IRS2: now also DEVICE1.P0.6, J6.2; no longer DEVICE1.P2.2/SW1, J6.7
- net IRS4: now also DEVICE1.P0.4/SAR0, J6.4; no longer J6.5
- net IRS6: now also DEVICE1.P0.2/SAR1, J6.6; no longer DEVICE1.P2.6, J6.3
- net IRS7: now also DEVICE1.P0.1, J6.7; no longer DEVICE1.P2.7, J6.2
- net IRS8: now also DEVICE1.P0.0, J6.8; no longer J6.1
- net LEDON: now also DEVICE1.P3.7; no longer DEVICE1.P2.0
- net N$10: now also DEVICE1.P2.4, J8.6; no longer DEVICE1.P0.4/SAR0, SV8.6
- net N$11: now also DEVICE1.P2.6, J8.5; no longer DEVICE1.P0.3/EXT_REF0, SV8.11
- net N$12: now also DEVICE1.P2.5, J8.4; no longer DEVICE1.P0.2/SAR1, SV8.12
- net N$8: now also DEVICE1.P2.1/LED1, J8.12; no longer DEVICE1.P0.6, SV8.4
- net N$9: now also DEVICE1.P2.0, J8.11; no longer DEVICE1.P0.5, SV8.5
- net SW1: now also S4.2; no longer S2.1
- net VCC: now also J5.1, J8.2, S4.1; no longer J5.3, S2.2, SV8.2
Other:
- board size 160 x 100 mm -> 137 x 79 mm

Commit message: eagle
schema klaar, nu pcb nog
Parts:
- removed S3: (no value), switch-dil:DS-01
- removed S4: (no value), SparkFun-Switches:SWITCH_SPDT_PTH_11.6X4.0MM
- added J9: Connector HC-05, SparkFun-Connectors:1X06_LOCK
- added S2: MOMENTARY-SWITCH-SPST-PTH-6.0MM, SparkFun-Switches:TACTILE_SWITCH_PTH_6.0MM
- added U$1, U$2: CONN_26, SparkFun-Connectors:1X26
- added U$3: SWITCH_GOTRON, SparkFun-Switches:SWITCH_SPDT_PTH_11.6X5.60MM
- LED1, LED2, LED3, LED4, LED5: value (none) -> 3.3V
- S1: value (none) -> MOMENTARY-SWITCH-SPST-PTH-6.0MM; device switch-dil:DS-01 -> SparkFun-Switches:TACTILE_SWITCH_PTH_6.0MM
- moved S1 11.0 mm to (70.0, 18.0), turned to 0 degrees
Connections:
- removed net ECHO1: DEVICE1.P12.3, J1.3
- removed net ECHO2: DEVICE1.P12.1/I2C(SDA), J2.3
- removed net ECHO3: DEVICE1.P1.0/SWDIO, J3.3
- removed net ENA: DEVICE1.P1.2, J4.8
- removed net ENB: DEVICE1.P1.7, J4.3
- removed net IN1: DEVICE1.P1.3, J4.7
- removed net IN2: DEVICE1.P1.4, J4.6
- removed net IN3: DEVICE1.P1.5, J4.5
- removed net IN4: DEVICE1.P1.6, J4.4
- removed net IRS1: DEVICE1.P0.7, J6.1
- removed net IRS2: DEVICE1.P0.6, J6.2
- removed net IRS3: DEVICE1.P0.5, J6.3
- removed net IRS4: DEVICE1.P0.4/SAR0, J6.4
- removed net IRS5: DEVICE1.P0.3/EXT_REF0, J6.5
- removed net IRS6: DEVICE1.P0.2/SAR1, J6.6
- removed net IRS7: DEVICE1.P0.1, J6.7
- removed net IRS8: DEVICE1.P0.0, J6.8
- removed net LED1: DEVICE1.P3.0, LED1.A
- removed net LED2: DEVICE1.P3.1, LED2.A
- removed net LED3: DEVICE1.P3.2, LED3.A
- removed net LED4: DEVICE1.P3.3, LED4.A
- removed net LED5: DEVICE1.P3.4, LED5.A
- removed net LEDON: DEVICE1.P3.7, J5.2
- removed net N$10: DEVICE1.P2.4, J8.6
- removed net N$11: DEVICE1.P2.6, J8.5
- removed net N$12: DEVICE1.P2.5, J8.4
- removed net N$13: J7.2, S3.1
- removed net N$14: J7.1, S3.2
- removed net N$8: DEVICE1.P2.1/LED1, J8.12
- removed net N$9: DEVICE1.P2.0, J8.11
- removed net SW1: DEVICE1.P3.5, S4.2
- removed net SW2: DEVICE1.P3.6, S1.1
- removed net TRIG1: DEVICE1.P12.2, J1.2
- removed net TRIG2: DEVICE1.P12.0/I2C(SCL), J2.2
- removed net TRIG3: DEVICE1.P1.1/SWDCLK, J3.2
- new net P0.0: DEVICE1.P0.0, J6.8, U$2.16
- new net P0.1: DEVICE1.P0.1, J6.7, U$2.17
- new net P0.2: DEVICE1.P0.2/SAR1, J6.6, U$2.18
- new net P0.3: DEVICE1.P0.3/EXT_REF0, J6.5, U$2.19
- new net P0.4: DEVICE1.P0.4/SAR0, J6.4, U$2.20
- new net P0.5: DEVICE1.P0.5, J6.3, U$2.21
- new net P0.6: DEVICE1.P0.6, J6.2, U$2.22
- new net P0.7: DEVICE1.P0.7, J6.1, U$2.23
- new net P1.0: DEVICE1.P1.0/SWDIO, J3.3, U$1.10
- new net P1.1: DEVICE1.P1.1/SWDCLK, J3.2, U$1.9
- new net P1.2: DEVICE1.P1.2, J4.8, U$1.8
- new net P1.3: DEVICE1.P1.3, J4.7, U$1.7
- new net P1.4: DEVICE1.P1.4, J4.6, U$1.6
- new net P1.5: DEVICE1.P1.5, J4.5, U$1.5
- new net P1.6: DEVICE1.P1.6, J4.4, U$1.4
- new net P1.7: DEVICE1.P1.7, J4.3, U$1.3
- new net P12.0: DEVICE1.P12.0/I2C(SCL), J2.2, U$1.11
- new net P12.1: DEVICE1.P12.1/I2C(SDA), J2.3, U$1.12
- new net P12.2: DEVICE1.P12.2, J1.2, U$1.13
- new net P12.3: DEVICE1.P12.3, J1.3, U$1.14
- new net P12.4: DEVICE1.P12.4, J9.1, U$1.15
- new net P12.5: DEVICE1.P12.5, J9.6, U$1.16
- new net P12.6: DEVICE1.P12.6/UARTRX, J9.5, U$1.17
- new net P12.7: DEVICE1.P12.7/UARTTX, J9.4, U$1.18
- new net P15.0: DEVICE1.P15.0, U$2.10
- new net P15.1: DEVICE1.P15.1, U$2.11
- new net P15.2: DEVICE1.P15.2/XTAL_OUT, U$2.12
- new net P15.3: DEVICE1.P15.3/XTAL_IN, U$2.13
- new net P15.4: DEVICE1.P15.4/CMOD, U$2.14
- new net P15.5: DEVICE1.P15.5, U$2.15
- new net P2.0: DEVICE1.P2.0, J8.11, U$1.26
- new net P2.1: DEVICE1.P2.1/LED1, J8.12, U$1.25
- new net P2.2: DEVICE1.P2.2/SW1, J8.13, U$1.24
- new net P2.3: DEVICE1.P2.3, J8.14, U$1.23
- new net P2.4: DEVICE1.P2.4, J8.6, U$1.22
- new net P2.5: DEVICE1.P2.5, J8.4, U$1.21
- new net P2.6: DEVICE1.P2.6, J8.5, U$1.20
- new net P2.7: DEVICE1.P2.7, U$1.19
- new net P3.0: DEVICE1.P3.0, LED1.A, U$2.2
- new net P3.1: DEVICE1.P3.1, LED2.A, U$2.3
- new net P3.2: DEVICE1.P3.2, LED3.A, U$2.4
- new net P3.3: DEVICE1.P3.3, LED4.A, U$2.5
- new net P3.4: DEVICE1.P3.4, LED5.A, U$2.6
- new net P3.5: DEVICE1.P3.5, S1.1, U$2.7
- new net P3.6: DEVICE1.P3.6, S2.1, U$2.8
- new net P3.7: DEVICE1.P3.7, J5.2, U$2.9
- new net RESET: DEVICE1.RESET, U$2.24
- new net VDDIO: DEVICE1.VDDIO, U$1.1
- net GND: now also J9.3, U$1.2, U$2.1, U$2.25; no longer S4.3
- net N$1: now also J7.2, U$3.2; no longer DEVICE1.P2.3, J8.14
- net N$7: now also J7.1, U$3.3; no longer DEVICE1.P2.2/SW1, J8.13
- net VCC: now also J9.2, S1.3, S2.3, U$2.26; no longer S1.2, S4.1

Commit message: eagle
pcb bijna af
Parts:
- removed J8: Connector LCD, SparkFun-Connectors:1X20
- moved U$3 115.0 mm to (7.00, 9.00)
- moved J7 115.0 mm to (15.7, 3.61)
- moved J9 85.1 mm to (96.0, 56.0), turned to 180 degrees
- moved J3 29.1 mm to (51.8, 55.9)
- moved J2 28.3 mm to (66.8, 55.9)
- moved J1 25.8 mm to (101.6, 49.1), turned to 270 degrees
- moved U$1 25.4 mm to (31.3, 44.9)
- moved U$2 24.4 mm to (31.3, 15.3)
- moved DEVICE1 24.0 mm to (47.8, 30.0)
- moved J4 23.0 mm to (22.8, 55.9)
- moved LED2 17.7 mm to (34.7, 8.97), turned to 0 degrees
- moved LED1 17.7 mm to (28.1, 8.97), turned to 0 degrees
- moved LED3 17.7 mm to (41.3, 8.97), turned to 0 degrees
- moved LED5 17.7 mm to (54.6, 8.97), turned to 0 degrees
- moved LED4 17.7 mm to (47.9, 8.97), turned to 0 degrees
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Connections:
- net GND: no longer J8.1, J8.3
- net P2.0: no longer J8.11
- net P2.1: no longer J8.12
- net P2.2: no longer J8.13
- net P2.3: no longer J8.14
- net P2.4: no longer J8.6
- net P2.5: no longer J8.4
- net P2.6: no longer J8.5
- net VCC: no longer J8.2
Routing:
- net VCC: track 0.00 -> 198.8 mm
- net P12.2: track 0.00 -> 57.0 mm
- net P3.7: track 0.00 -> 48.2 mm
- net P12.3: track 0.00 -> 47.2 mm
- net P0.0: track 0.00 -> 46.0 mm
- net P0.1: track 0.00 -> 40.5 mm
- net P12.4: track 0.00 -> 38.5 mm
- net P0.2: track 0.00 -> 36.4 mm
- net P0.5: track 0.00 -> 34.3 mm
- net P0.3: track 0.00 -> 33.4 mm
- net P0.6: track 0.00 -> 32.4 mm
- net P3.6: track 0.00 -> 31.1 mm
- net P0.4: track 0.00 -> 31.0 mm
- net P3.5: track 0.00 -> 25.2 mm
- net P12.5: track 0.00 -> 24.8 mm
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- added copper zone on layer 1, net GND
Other:
- board size 137 x 79 mm -> 106 x 60 mm
- board text added: "MADE BY HUMANS"
- board text added: "ON EARTH"
