File: Eagle/SchemaRobotV1.0.sch (EAGLE design)
At the start: 24 parts, among them J1 Connector US1, J2 Connector US 2, J3 Connector US 2, J4 Connector H-Brug, J5 Connector IR voeding, J6 Connector IR signalen, J7 Connector batterij 12v, J9 Connector HC-05

Commit message: eagle
meer padjes van top naar bottom
Connections:
- net GND: now also S1.2, S2.2
- net VCC: no longer S1.2, S2.2
Changed lines of the file:
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@@
 <part name="S1" library="SchemaRobotV1.0" deviceset="SPARKFUN-SWITCHES_MOMENTARY-SWITCH-SPST" device="-PTH-6.0MM"/>
 <part name="S2" library="SchemaRobotV1.0" deviceset="SPARKFUN-SWITCHES_MOMENTARY-SWITCH-SPST" device="-PTH-6.0MM"/>
-<part name="P+5" library="supply1" library_urn="urn:adsk.eagle:library:371" deviceset="VCC" device=""/>
 <part name="U$3" library="SchemaRobotV1.0" deviceset="SPARKFUN-SWITCHES_SWITCH_GOTRON" device=""/>
+<part name="GND2" library="supply1" library_urn="urn:adsk.eagle:library:371" deviceset="GND" device=""/>
 </parts>
 <sheets>
@@
 <instance part="S1" gate="G$1" x="157.48" y="81.28"/>
 <instance part="S2" gate="G$1" x="157.48" y="88.9"/>
-<instance part="P+5" gate="VCC" x="170.18" y="99.06" rot="MR0"/>
 <instance part="U$3" gate="G$1" x="66.04" y="15.24"/>
+<instance part="GND2" gate="1" x="170.18" y="73.66"/>
 </instances>
 <busses>
@@
 <label x="12.7" y="124.46" size="1.778" layer="95"/>
 </segment>
+<segment>
+<pinref part="S2" gate="G$1" pin="2"/>
+<wire x1="162.56" y1="88.9" x2="170.18" y2="88.9" width="0.1524" layer="91"/>
+<pinref part="S1" gate="G$1" pin="2"/>
+<wire x1="162.56" y1="81.28" x2="170.18" y2="81.28" width="0.1524" layer="91"/>
+<wire x1="170.18" y1="81.28" x2="170.18" y2="88.9" width="0.1524" layer="91"/>
+<pinref part="GND2" gate="1" pin="GND"/>
+<wire x1="170.18" y1="81.28" x2="170.18" y2="76.2" width="0.1524" layer="91"/>
+<junction x="170.18" y="81.28"/>
+</segment>
 </net>
 <net name="VCC" class="0">
@@
 <pinref part="P+4" gate="VCC" pin="VCC"/>
 </segment>
-<segment>
-<pinref part="S2" gate="G$1" pin="2"/>
-<wire x1="162.56" y1="88.9" x2="170.18" y2="88.9" width="0.1524" layer="91"/>
-<wire x1="170.18" y1="88.9" x2="170.18" y2="96.52" width="0.1524" layer="91"/>
-<pinref part="S1" gate="G$1" pin="2"/>
-<wire x1="162.56" y1="81.28" x2="170.18" y2="81.28" width="0.1524" layer="91"/>
-<wire x1="170.18" y1="81.28" x2="170.18" y2="88.9" width="0.1524" layer="91"/>
-<junction x="170.18" y="88.9"/>
-<pinref part="P+5" gate="VCC" pin="VCC"/>
-</segment>
-</net>
+</net>

Commit message: eagle
padjes verbeterd
Parts:
- LED2: device led:LED5MM -> SchemaRobotV1.0:LED_LED5MM
Changed lines of the file:
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@@
 <part name="R5" library="SchemaRobotV1.0" deviceset="EAGLE-LTSPICE_R" device="0204/7" value="100 ohm"/>
 <part name="LED1" library="SchemaRobotV1.0" deviceset="LED_LED" device="5MM" value="3.3V"/>
-<part name="LED2" library="led" library_urn="urn:adsk.eagle:library:259" deviceset="LED" device="5MM" package3d_urn="urn:adsk.eagle:package:15799/2" value="3.3V"/>
+<part name="LED2" library="SchemaRobotV1.0" deviceset="LED_LED" device="5MM" value="3.3V"/>
 <part name="LED3" library="SchemaRobotV1.0" deviceset="LED_LED" device="5MM" value="3.3V"/>
 <part name="LED4" library="SchemaRobotV1.0" deviceset="LED_LED" device="5MM" value="3.3V"/>
@@
 will not be understood (or retained) with this version.
 </note>
-<note version="8.3" severity="warning">
-Since Version 8.3, EAGLE supports the association of 3D packages
-with devices in libraries, schematics, and board files. Those 3D
-packages will not be understood (or retained) with this version.
-</note>
 </compatibility>
