File: Schema's/Eagle/SchemaRobotV1.0.brd (EAGLE design)
At the start: 106 x 60 mm, 24 parts, among them J1 Connector US1, J2 Connector US 2, J3 Connector US 2, J4 Connector H-Brug, J5 Connector IR voeding, J6 Connector IR signalen, J7 Connector batterij 12v, J9 Connector HC-05

Commit message: roadster
ITS ALIVE
Parts:
- J3: value Connector US 2 -> Connector US 3
Changed lines of the file:
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@@
 <attribute name="SF_ID" value="2xPRT-08084" x="67.57" y="55.63" size="1.778" layer="27" display="off"/>
 </element>
-<element name="J3" library="SchemaRobotV1.0" package="SPARKFUN-CONNECTORS_SCREWTERMINAL-3.5MM-4" value="Connector US 2" x="52.8" y="55.73">
+<element name="J3" library="SchemaRobotV1.0" package="SPARKFUN-CONNECTORS_SCREWTERMINAL-3.5MM-4" value="Connector US 3" x="52.8" y="55.73">
 <attribute name="PROD_ID" value="2xCONN-08399" x="52.8" y="55.73" size="1.778" layer="27" display="off"/>
 <attribute name="SF_ID" value="2xPRT-08084" x="52.8" y="55.73" size="1.778" layer="27" display="off"/>
