File: Schema's/Eagle/SchemaRobotV1.0.sch (EAGLE design)
At the start: 24 parts, among them J1 Connector US1, J2 Connector US 2, J3 Connector US 2, J4 Connector H-Brug, J5 Connector IR voeding, J6 Connector IR signalen, J7 Connector batterij 12v, J9 Connector HC-05

Commit message: roadster
ITS ALIVE
Parts:
- J3: value Connector US 2 -> Connector US 3
Changed lines of the file:
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@@
 <part name="J1" library="SchemaRobotV1.0" deviceset="SPARKFUN-CONNECTORS_CONN_04" device="SCREW" value="Connector US1"/>
 <part name="J2" library="SchemaRobotV1.0" deviceset="SPARKFUN-CONNECTORS_CONN_04" device="SCREW" value="Connector US 2"/>
-<part name="J3" library="SchemaRobotV1.0" deviceset="SPARKFUN-CONNECTORS_CONN_04" device="SCREW" value="Connector US 2"/>
+<part name="J3" library="SchemaRobotV1.0" deviceset="SPARKFUN-CONNECTORS_CONN_04" device="SCREW" value="Connector US 3"/>
 <part name="J4" library="SchemaRobotV1.0" deviceset="SPARKFUN-CONNECTORS_CONN_08" device="3.5MM-8" value="Connector H-Brug"/>
 <part name="J5" library="SchemaRobotV1.0" deviceset="SPARKFUN-CONNECTORS_CONN_04" device="SCREW" value="Connector IR voeding"/>
